Commit message: feat: Add static camera link and joint to multiagent simulation models

File: src/multiagent_simulation/models/camera/model.xacro (robot description, xacro)
@@ -18,7 +18,22 @@
       </inertial>
     </link>
+    <link name="cameras_static_link">
+      <pose>0 0 0 0 0 0</pose>
+      <kinematic>true</kinematic>
+      <gravity>false</gravity>
+      <inertial>
+        <mass>0.0</mass>
+        <inertia>
+          <ixx>0.0</ixx>
+          <ixy>0.0</ixy>
+          <iyy>0.0</iyy>
+          <iyz>0.0</iyz>
+          <izz>0.0</izz>
+        </inertia>
+      </inertial>
+    </link>
     <!-- Macro Definition for Camera -->
     <xacro:macro name="camera_sensor"
-      params="name pose optical_pose horizontal_fov image_width image_height update_rate format intrinsics:='277 277 160 120' distortion:='0.0 0.0 0.0 0.0'">
+      params="name pose optical_pose horizontal_fov image_width image_height update_rate format parent_link:='cameras_link' intrinsics:='277 277 160 120' distortion:='0.0 0.0 0.0 0.0'">
       <xacro:property name="fx" value="${intrinsics.split()[0]}" />
       <xacro:property name="fy" value="${intrinsics.split()[1]}" />
@@ -123,5 +138,5 @@
       </joint>
       <joint name="${name}_joint" type="fixed">
-        <parent>cameras_link</parent>
+        <parent>${parent_link}</parent>
         <child>${name}_link</child>
         <preserve_fixed_joint>true</preserve_fixed_joint>
@@ -155,4 +170,5 @@
       optical_pose="0.0 -0.02 -0.05 0 3.14 1.57"
       horizontal_fov="0.92729343"
+      parent_link="cameras_static_link"
       intrinsics="960.0 960.0 564.0 564.0"
       distortion="-0.15 0.03 0.001 0.001"
@@ -166,4 +182,5 @@
       optical_pose="-0.05 -0.02 -0.05 0 3.14 1.57"
       horizontal_fov="1.448"
+      parent_link="cameras_static_link"
       intrinsics="471.42701287242807 470.7784450086591 389.70874283839333 258.6696297186715"
       distortion="-0.3141061887234863 0.12230478626307012 -0.00010883202540227276 -0.0003551641298941904"
